File: nvim-coaster.kicad_pcb (KiCad board)
At the start: 2 copper layers, 207.1 x 99.3 mm, 0 parts

Commit message: changes
Other:
- board size 207.1 x 99.3 mm -> 99.1 x 99.1 mm
- board text added: "neovim"
- board text removed: "0 last yank {dblquote} unnamed register, last delete or yank % current file name # alternate file name * clipboard contents + clipboard contents / last search pattern : last command . last inserted text - last small delete = expression register _ black hole register"
- board text removed: ":reg show register content {dblquote}xy yank to register x {dblquote}xp paste from register x {dblquote}+y yank to system clipboard {dblquote}+p paste from system clipboard"
- board text removed: ":vim[grep] /pattern/ {`{file}`} e.g. :vim[grep] /foo/ **/* :cn jump to next match :cp jump to previous match :copen open a window containing list of matches :cclose close the quickfix window"
- board text removed: "Movement"
- board text removed: "Registers"
- board text removed: "Search multiple files"
- board text removed: "Special registers"
- board text removed: "h left (pointer finger) j down (pointer finger) k up (middle finger) l right (ring finger) gj down multi line gk up multi line H top of screen M middle of screen L bottom of screen w word forward (start) W word forward (start) incl. punctuation e word forward (end) E word forward (end) incl. punctuation b word backward (start) B word backward (start) incl. punctuation ge word backward (end) gE wo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"

Commit message: First version ready
Other:
- board text added: "0 {dblquote} % # * + / : . - = _"
- board text added: ":reg {dblquote}xy {dblquote}xp {dblquote}+y {dblquote}+p"
- board text added: ":tabnew Ctrl+wT gt or :tabn[ext] gT or :tabp[revious] #gt :tabm[ove] # :tabc[lose] :tabo[nly] :tabdo cmd"
- board text added: ":vim[grep] /pattern/ {`{file}`} e.g. :vim[grep] /foo/ **/* :cn :cp :copen :cclose"
- board text added: "Movement"
- board text added: "Registers"
- board text added: "Search multiple files"
- board text added: "Special registers"
- board text added: "Tabs"
- board text added: "h j k l gj gk H M L w W e E b B ge gE % 0 ^ $ g_ gg G gd gD fx tx Fx Tx ; , } {brace} zz zt zb"
- board text added: "jump to next match jump to previous match open a window containing list of matches close the quickfix window"
- board text added: "last yank unnamed register, last delete or yank current file name alternate file name clipboard contents clipboard contents last search pattern last command last inserted text last small delete expression register black hole register"
- board text added: "left down up right down multi line up multi line top of screen middle of screen bottom of screen word forward (start) word forward (start) incl. punctuation word forward (end) word forward (end) incl. punctuation word backward (start) word backward (start) incl. punctuation word backward (end) word backward (end) incl. punctuation move to matching (), {brace}, [] start of line first non blank cha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"
- board text added: "open a file in a new tab move the current window to a new tab move to the next tab move to the previous tab move to the tab number # move current tab to the #th position close the current tab close all except the current tab run the command cmd on all tabs"
- board text added: "show register content yank to register x paste from register x yank to system clipboard paste from system clipboard"
Changed lines of the file:
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@@
       (xy 48.505761 49.075415)
     ) (layer "F.Cu") (width 0) (fill solid))
+  (gr_poly
+    (pts
+      (xy 120.809097 51.451434)
+      (xy 120.792264 58.040472)
+      (xy 121.216205 58.5013)
+      (xy 123.300513 55.36277)
+      (xy 123.300513 48.944551)
+    ) (layer "B.Cu") (width 0) (fill solid))
+  (gr_poly
+    (pts
+      (xy 121.418588 58.737127)
+      (xy 123.208897 60.52799)
+      (xy 129.610087 50.783472)
+      (xy 127.81643 48.970991)
+    ) (layer "B.Cu") (width 0) (fill solid))
+  (gr_poly
+    (pts
+      (xy 127.85 54.054718)
+      (xy 127.85 60.5)
+      (xy 130.310625 58.04258)
+      (xy 130.310625 51.426442)
+      (xy 129.895241 51.006751)
+    ) (layer "B.SilkS") (width 0) (fill solid))
+  (gr_line (start 71.4 73.3) (end 88.3 73.3) (layer "B.SilkS") (width 0.15))
+  (gr_line (start 80.25 114.5) (end 88.15 114.5) (layer "B.SilkS") (width 0.15))
+  (gr_line (start 112.45 69.4) (end 130.65 69.4) (layer "B.SilkS") (width 0.15))
+  (gr_line (start 48.5 55.3) (end 88.1 55.3) (layer "B.SilkS") (width 0.15))
+  (gr_line (start 56.8 87.5) (end 88.5 87.5) (layer "B.SilkS") (width 0.15))
   (gr_line locked (start 85.2 51.3) (end 96.5 51.3) (layer "F.SilkS") (width 0.15))
   (gr_line locked (start 45.35 128.6) (end 71.65 128.6) (layer "F.SilkS") (width 0.15))
@@
   (gr_line locked (start 45.612104 109.6) (end 57.912104 109.6) (layer "F.SilkS") (width 0.15))
   (gr_line locked (start 86.1 132.3) (end 98.6 132.3) (layer "F.SilkS") (width 0.15))
+  (gr_poly
+    (pts
+      (xy 121.452376 58.725012)
+      (xy 123.242685 60.515875)
+      (xy 129.643875 50.771357)
+      (xy 127.850218 48.958876)
+    ) (layer "B.Mask") (width 0) (fill solid))
+  (gr_poly
+    (pts
+      (xy 120.802459 51.449884)
+      (xy 120.785626 58.038922)
+      (xy 121.209567 58.49975)
+      (xy 123.293875 55.36122)
+      (xy 123.293875 48.943001)
+    ) (layer "B.Mask") (width 0) (fill solid))
   (gr_poly locked
     (pts
@@
     (effects (font (size 2.5 2.5) (thickness 0.6)))
   )
+  (gr_text "neovim" (at 106.122191 57.595576) (layer "B.Cu")
+    (effects (font (size 5 5) (thickness 0.15)) (justify mirror))
+  )
+  (gr_text "Registers" (at 79.9 71) (layer "B.Cu")
+    (effects (font (size 2.5 2.5) (thickness 0.6)) (justify mirror))
+  )
+  (gr_text "Tabs" (at 84.25 112.1) (layer "B.Cu")
+    (effects (font (size 2.5 2.5) (thickness 0.6)) (justify mirror))
+  )
+  (gr_text "Special registers" (at 72.8 85.3) (layer "B.Cu")
+    (effects (font (size 2.5 2.5) (thickness 0.6)) (justify mirror))
+  )
+  (gr_text "Movement" (at 121.75 67.1) (layer "B.Cu")
+    (effects (font (size 2.5 2.5) (thickness 0.6)) (justify mirror))
+  )
+  (gr_text "Search multiple files" (at 68.2 52.8) (layer "B.Cu")
+    (effects (font (size 2.5 2.5) (thickness 0.6)) (justify mirror))
+  )
+  (gr_text "jump to next match\njump to previous match\nopen a window containing list of matches\nclose the quickfix window" (at 80.5 63.8) (layer "B.SilkS")
+    (effects (font (size 1 1) (thickness 0.15)) (justify left mirror))
+  )
+  (gr_text ":vim[grep] /pattern/ {`{file}`}\ne.g. :vim[grep] /foo/ **/*\n\n:cn	   \n:cp	   \n:copen \n:cclose" (at 88.3 61.5) (layer "B.SilkS")
+    (effects (font (size 1 1) (thickness 0.15)) (justify left mirror))
+  )
+  (gr_text "h \nj \nk \nl \ngj\ngk\nH \nM \nL \nw \nW \ne \nE \nb \nB \nge\ngE\n% \n0 \n^ \n$ \ng_\ngg\nG \ngd\ngD\nfx\ntx\nFx\nTx\n; \n, \n} \n{brace}\nzz\nzt\nzb" (at 130.7 100.2) (layer "B.SilkS")
+    (effects (font (size 1 1) (thickness 0.15)) (justify left mirror))
+  )
+  (gr_text "0\n{dblquote}\n%\n#\n*\n+\n/\n:\n.\n-\n=\n_" (at 88.7 98.4) (layer "B.SilkS")
+    (effects (font (size 1 1) (thickness 0.15)) (justify left mirror))
+  )
+  (gr_text "open a file in a new tab\nmove the current window to a new tab\nmove to the next tab\nmove to the previous tab\nmove to the tab number #\nmove current tab to the #th position\nclose the current tab\nclose all except the current tab\nrun the command cmd on all tabs\n" (at 72 124.2) (layer "B.SilkS")
+    (effects (font (size 1 1) (thickness 0.15)) (justify left mirror))
+  )
+  (gr_text "left\ndown\nup\nright\ndown multi line\nup multi line\ntop of screen\nmiddle of screen\nbottom of screen\nword forward (start)\nword forward (start) incl. punctuation\nword forward (end)\nword forward (end) incl. punctuation\nword backward (start)\nword backward (start) incl. punctuation\nword backward (end)\nword backward (end) incl. punctuation\nmove to matching (), {brace}, []\nstart of line\nfirst non blank char\nend of line\nlast non-blank char of the line\nfirst line\nlast line\nmove to local declaration\nmove to global declaration\nnext occurence of char x\nbefore next occurence of char x\nprevious occurence of char x\nbefore previous occurence of char x\nrepeat previous f, t, F or T\nrepeat previous f, t, F or T backwards\nnext paragraph\nprevious paragraph\ncenter cursor on screen\ncursor to top\ncursor to bottom" (at 127.5 100.2) (layer "B.SilkS")
+    (effects (font (size 1 1) (thickness 0.15)) (justify left mirror))
+  )
+  (gr_text ":reg\n{dblquote}xy	\n{dblquote}xp	\n{dblquote}+y\n{dblquote}+p" (at 88.4 77.4) (layer "B.SilkS")
+    (effects (font (size 1 1) (thickness 0.15)) (justify left mirror))
+  )
+  (gr_text ":tabnew       \nCtrl+wT       \ngt  or :tabn[ext]    \ngT or :tabp[revious]\n#gt           \n:tabm[ove] #  \n:tabc[lose]   \n:tabo[nly]    \n:tabdo cmd    \n" (at 88.65 124.2) (layer "B.SilkS")
+    (effects (font (size 1 1) (thickness 0.15)) (justify left mirror))
+  )
+  (gr_text "show register content\nyank to register x\npaste from register x\nyank to system clipboard\npaste from system clipboard" (at 84.1 77.4) (layer "B.SilkS")
+    (effects (font (size 1 1) (thickness 0.15)) (justify left mirror))
+  )
+  (gr_text "last yank\nunnamed register, last delete or yank\ncurrent file name\nalternate file name\nclipboard contents\nclipboard contents\nlast search pattern\nlast command\nlast inserted text\nlast small delete\nexpression register\nblack hole register" (at 86.3 98.5) (layer "B.SilkS")
+    (effects (font (size 1 1) (thickness 0.15)) (justify left mirror))
+  )
   (gr_text "yy		yank (copy) line\nyw		yank word\nyiw		yank word under cursor\nyaw		yank word under cursor including next whitespace\nY		yank to end of line\np		put (paste)	after cursor\nP		put before cursor\ngp		put after cursor and leave cursor after the new text\ngP		put before cursor and leave cursor after the new text\nx		delete (cut) character\nD		delete to the end of line\ndd		delete a line\ndw		delete word\ndiw		delete word under cursor\ndaw		delete word under cursor including next whitespace\n:3,5d	delete lines 3, 4 and 5\n\n:g/foo/d	delete all lines containing foo\n:g!/foo/d	delete all liens not containing foo" (at 85.9 111.5) (layer "F.SilkS")
     (effects (font (size 1 1) (thickness 0.15)) (justify left))
@@
     (effects (font (size 1 1) (thickness 0.15)) (justify left))
   )
+  (gr_text "neovim" (at 106.122191 57.595576) (layer "B.Mask")
+    (effects (font (size 5 5) (thickness 0.15)) (justify mirror))
+  )
+  (gr_text "Movement" (at 121.75 67.1) (layer "B.Mask")
+    (effects (font (size 2.5 2.5) (thickness 0.6)) (justify mirror))
+  )
+  (gr_text "Registers" (at 79.9 71) (layer "B.Mask")
+    (effects (font (size 2.5 2.5) (thickness 0.6)) (justify mirror))
+  )
+  (gr_text "Search multiple files" (at 68.2 52.8) (layer "B.Mask")
+    (effects (font (size 2.5 2.5) (thickness 0.6)) (justify mirror))
+  )
+  (gr_text "Tabs" (at 84.25 112.1) (layer "B.Mask")
+    (effects (font (size 2.5 2.5) (thickness 0.6)) (justify mirror))
+  )
+  (gr_text "Special registers" (at 72.8 85.3) (layer "B.Mask")
+    (effects (font (size 2.5 2.5) (thickness 0.6)) (justify mirror))
+  )
   (gr_text "Indent" (at 90.6 49.2) (layer "F.Mask")
